File: Hardware/V1/UniAdapter.sch (EAGLE design)
At the start: 24 parts, among them IC1 LD1117S33TR, IC2 SN65HVD232D, IC3 STM32F072CBT6, X1 CAN Bus, X2 CAN Bus

Commit message: Revert "Revert "AnySense 1.1""
This reverts commit 477dbe3a037d16c593f52677c37ec78f086be774.
Parts:
- LD1: OC_FARNELL (none) -> 2099221
- LD2: OC_FARNELL (none) -> 2099223
- R4: value 55Ohm -> 68Ohm; OC_FARNELL (none) -> 2331710
- R5: value 55Ohm -> 56Ohm; OC_FARNELL (none) -> 2331709
Changed lines of the file:
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@@
 </part>
 <part name="P+4" library="supply1" deviceset="VCC" device=""/>
-<part name="R4" library="rcl" deviceset="R-EU_" device="R0603" value="55Ohm"/>
-<part name="R5" library="rcl" deviceset="R-EU_" device="R0603" value="55Ohm"/>
-<part name="LD1" library="led" deviceset="LED" device="CHIPLED_0603" value="RED"/>
-<part name="LD2" library="led" deviceset="LED" device="CHIPLED_0603" value="GREEN"/>
+<part name="R4" library="rcl" deviceset="R-EU_" device="R0603" value="68Ohm">
+<attribute name="OC_FARNELL" value="2331710"/>
+</part>
+<part name="R5" library="rcl" deviceset="R-EU_" device="R0603" value="56Ohm">
+<attribute name="OC_FARNELL" value="2331709"/>
+</part>
+<part name="LD1" library="led" deviceset="LED" device="CHIPLED_0603" value="RED">
+<attribute name="OC_FARNELL" value="2099221"/>
+</part>
+<part name="LD2" library="led" deviceset="LED" device="CHIPLED_0603" value="GREEN">
+<attribute name="OC_FARNELL" value="2099223"/>
+</part>
 <part name="GND5" library="supply1" deviceset="GND" device=""/>
 </parts>
@@
 </instance>
 <instance part="P+4" gate="VCC" x="68.58" y="-63.5"/>
-<instance part="R4" gate="G$1" x="111.76" y="30.48"/>
-<instance part="R5" gate="G$1" x="111.76" y="20.32"/>
-<instance part="LD1" gate="G$1" x="127" y="30.48" rot="R90"/>
-<instance part="LD2" gate="G$1" x="127" y="20.32" rot="R90"/>
+<instance part="R4" gate="G$1" x="111.76" y="30.48">
+<attribute name="OC_FARNELL" x="111.76" y="30.48" size="1.778" layer="96" display="off"/>
+</instance>
+<instance part="R5" gate="G$1" x="111.76" y="20.32">
+<attribute name="OC_FARNELL" x="111.76" y="20.32" size="1.778" layer="96" display="off"/>
+</instance>
+<instance part="LD1" gate="G$1" x="127" y="30.48" rot="R90">
+<attribute name="OC_FARNELL" x="127" y="30.48" size="1.778" layer="96" rot="R90" display="off"/>
+</instance>
+<instance part="LD2" gate="G$1" x="127" y="20.32" rot="R90">
+<attribute name="OC_FARNELL" x="127" y="20.32" size="1.778" layer="96" rot="R90" display="off"/>
+</instance>
 <instance part="GND5" gate="1" x="134.62" y="15.24"/>
 </instances>
@@
 <wire x1="132.08" y1="30.48" x2="134.62" y2="30.48" width="0.1524" layer="91"/>
 <wire x1="134.62" y1="30.48" x2="134.62" y2="20.32" width="0.1524" layer="91"/>
-</segment>
-</net>
+<junction x="134.62" y="20.32"/>
+</segment>
+</net>

Commit message: Order Codes changed, cream frame reduced, BOOT0 rerouted
Parts:
- R1: OC_FARNELL 2331740 -> 2059627
- R2, R3: OC_FARNELL 2331730 -> 2059608
- R4: OC_FARNELL 2331710 -> 2059570
- R5: OC_FARNELL 2331709 -> 2059568
Changed lines of the file:
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@@
 </part>
 <part name="R1" library="rcl" deviceset="R-EU_" device="R0603" value="10k">
-<attribute name="OC_FARNELL" value="2331740"/>
+<attribute name="OC_FARNELL" value="2059627"/>
 </part>
 <part name="GND2" library="supply1" deviceset="GND" device=""/>
@@
 <part name="X2" library="con-molex-micro-fit-3_0" deviceset="HEADER_POS4_?" device="43650-0412" value="CAN Bus"/>
 <part name="R3" library="rcl" deviceset="R-EU_" device="R0603" value="1.8K">
-<attribute name="OC_FARNELL" value="2331730"/>
+<attribute name="OC_FARNELL" value="2059608"/>
 </part>
 <part name="R2" library="rcl" deviceset="R-EU_" device="R0603" value="1.8K">
-<attribute name="OC_FARNELL" value="2331730"/>
+<attribute name="OC_FARNELL" value="2059608"/>
 </part>
 <part name="P+4" library="supply1" deviceset="VCC" device=""/>
 <part name="R4" library="rcl" deviceset="R-EU_" device="R0603" value="68Ohm">
-<attribute name="OC_FARNELL" value="2331710"/>
+<attribute name="OC_FARNELL" value="2059570"/>
 </part>
 <part name="R5" library="rcl" deviceset="R-EU_" device="R0603" value="56Ohm">
-<attribute name="OC_FARNELL" value="2331709"/>
+<attribute name="OC_FARNELL" value="2059568"/>
 </part>
 <part name="LD1" library="led" deviceset="LED" device="CHIPLED_0603" value="RED">
